File: Schematic/MCU.kicad_sch (KiCad schematic)
At the start: 27 parts, among them J101 USB_B_Micro, J102 Conn_02x05_Odd_Even, SW101 SW_SPST, U101 ESP32-S3-WROOM-1, U102 LMR50410-Q, U303 AMS1117

Commit message: Rev. 2 schematic and PCB
Parts:
- added C102: 2.2uF, Capacitor_SMD:C_0805_2012Metric, symbol Device:C
- C101, C102, C108, C109, C111: footprint Capacitor_THT:C_Disc_D4.7mm_W2.5mm_P5.00mm -> Capacitor_SMD:C_0805_2012Metric
- L101: value 3.3uH -> 4.7uH
- R101, R102: footprint PCM_Resistor_THT_AKL:R_Axial_DIN0207_L6.3mm_D2.5mm_P7.62mm_Horizontal -> PCM_Resistor_SMD_AKL:R_0805_2012Metric
- R103: value 47k -> 89k; footprint PCM_Resistor_THT_AKL:R_Axial_DIN0207_L6.3mm_D2.5mm_P7.62mm_Horizontal -> PCM_Resistor_SMD_AKL:R_0805_2012Metric
Connections:
- net +3.3V: now also C102.1; no longer C112.1, L101.2, R103.2
- net +5V: now also C112.1, L101.2, R103.2
- net ENCB_L: now also U101.6 (GPIO6/TOUCH6/ADC1_CH5); no longer U101.34 (MTDI/GPIO41/CLK_OUT1)
- net ENCB_R: now also U101.7 (GPIO7/TOUCH7/ADC1_CH6); no longer U101.33 (MTDO/GPIO40/CLK_OUT2)
- net ENCC_L: now also U101.8 (GPIO15/U0RTS/ADC2_CH4/XTAL_32K_P); no longer U101.6 (GPIO6/TOUCH6/ADC1_CH5)
- net ENCC_R: now also U101.9 (GPIO16/U0CTS/ADC2_CH5/XTAL_32K_N); no longer U101.32 (MTCK/GPIO39/CLK_OUT3/SUBSPICS1)
- net EXP_CS: now also U101.23 (GPIO21); no longer U101.38 (GPIO2/TOUCH2/ADC1_CH1)
- net EXP_RST: now also U101.17 (GPIO9/TOUCH9/ADC1_CH8/FSPIHD/SUBSPIHD); no longer U101.7 (GPIO7/TOUCH7/ADC1_CH6)
- net GND: now also C102.2
- net LDAC: now also U101.33 (MTDO/GPIO40/CLK_OUT2); no longer U101.17 (GPIO9/TOUCH9/ADC1_CH8/FSPIHD/SUBSPIHD)
- net PIXELS: now also U101.32 (MTCK/GPIO39/CLK_OUT3/SUBSPICS1); no longer U101.23 (GPIO21)
- net SCL: now also U101.10 (GPIO17/U1TXD/ADC2_CH6); no longer U101.11 (GPIO18/U1RXD/ADC2_CH7/CLK_OUT3)
- net SDA: now also U101.11 (GPIO18/U1RXD/ADC2_CH7/CLK_OUT3); no longer U101.10 (GPIO17/U1TXD/ADC2_CH6)
- net V_USB: now reaches D102.2 (A), J101.1 (VBUS)
- net EN: now reaches C101.1, R101.2, SW101.1 (A), U101.3 (EN)
- net IO19 renamed USB-
- net IO20 renamed USB+
Other:
- note added: "5v Buck Converter"
- note added: "Note: this output directly to 3.3v in rev. 1, hopefully less noise now going through the LDO"
- note removed: "3.3v Buck Converter"
- moved on the sheet: C110, C111, C112, L101, R102, R103, U102
