File: Schematic/IO.kicad_sch (KiCad schematic)
At the start: 87 parts, among them J201 CV1, J202 CV2, J203 CV3, J204 CV4, J205 GATE1, J206 GATE4, J207 GATE2, J208 GATE3, J209 Display, Q101 BC547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

Commit message: Output ISR
Parts:
- removed R229, R232, R235, R236, R237, R238, R239, R240, R241: 10k, PCM_Resistor_THT_AKL:R_Axial_DIN0207_L6.3mm_D2.5mm_P7.62mm_Horizontal, symbol Device:R_US
Connections:
- net at D218.4 (DOUT): now also D225.2 (DIN); no longer D222.4 (DOUT)

Commit message: Rev. 2 schematic and PCB
Parts:
- Q101: value BC547 -> BC847; footprint PCM_Package_TO_SOT_THT_AKL:TO-92L_HandSolder -> PCM_Package_TO_SOT_SMD_AKL:SOT-23; symbol PCM_Transistor_BJT_AKL:BC547 -> PCM_Transistor_BJT_AKL:BC847
- R104, R105, R106, R107, R108, R109, R110, R111, R112, R113, R114, R115, R116, R117, R118, R227, R228, R230, R231, R233, R234: footprint PCM_Resistor_THT_AKL:R_Axial_DIN0207_L6.3mm_D2.5mm_P7.62mm_Horizontal -> PCM_Resistor_SMD_AKL:R_0805_2012Metric
Connections:
- net C1: now also U201.4 (GPB3); no longer U201.6 (GPB5)
- net C1_GATE: now also Q101.3 (C); no longer Q101.1 (C)
- net C2: now also U201.3 (GPB2); no longer U201.7 (GPB6)
- net C2_GATE: now also Q101.3 (C); no longer Q101.1 (C)
- net C3: now also U201.2 (GPB1); no longer U201.8 (GPB7)
- net C3_GATE: now also Q101.3 (C); no longer Q101.1 (C)
- net C4: now also U201.1 (GPB0); no longer U201.21 (GPA0)
- net C4_GATE: now also Q101.3 (C); no longer Q101.1 (C)
- net ENCA_B: now also U201.7 (GPB6); no longer U201.1 (GPB0)
- net ENCB_B: now also U201.6 (GPB5); no longer U201.2 (GPB1)
- net ENCC_B: now also U201.5 (GPB4); no longer U201.3 (GPB2)
- net GND: now also Q101.2 (E), Q101.2 (E), Q101.2 (E), Q101.2 (E); no longer Q101.3 (E), Q101.3 (E), Q101.3 (E), Q101.3 (E)
- net PG_LEFT: now also U201.28 (GPA7); no longer U201.27 (GPA6)
- net PG_RIGHT: now also U201.27 (GPA6); no longer U201.28 (GPA7)
- net at R104.2: now also Q101.1 (B); no longer Q101.2 (B) (x4)

Commit message: PCB in git
Parts:
- added C102 (x3): 0.1uF, Capacitor_SMD:C_0805_2012Metric, symbol Device:C
Connections:
- net +12V: now also C102.1
- net +3.3V: now also C102.1
- net -12V: now also C102.1
- net GND: now also C102.2, C102.2, C102.2
Other:
- moved on the sheet: U104E
