File: Schematic/Ultra64_mk2.kicad_pcb (KiCad board)
At the start: 4 copper layers, 101.6 x 110 mm, 109 parts, among them J201 CV1, J202 CV2, J203 CV3, J204 CV4, J205 GATE1, J206 GATE4, J207 GATE2, J208 GATE3, J209 Display, J301 USB_B_Micro, J302 Conn_02x05_Odd_Even, Q201 BC847, Q202 BC847, Q203 BC847, Q204 BC847, SW201 RotaryEncoder_Switch, SW202 RotaryEncoder_Switch, SW203 RotaryEncoder_Switch, SW204 SW_SPST, SW205 SW_SPST, SW206 SW_SPST, SW207 SW_SPST, SW208 SW_SPST, SW209 SW_SPST, SW301 SW_SPST, SW302 SW_SPST, U201 MCP4728, U202 TL074, U203 MCP23S17_SO, U301 ESP32-S3-WROOM-1, U302 LMR50410-Q, U303 AMS1117

Commit message: fixed pins
Parts:
- moved U301 0.08 mm to (21.3, 88.1)
Routing:
- net DAC_RDY: track 105.6 -> 100.5 mm
- net SCL: track 88.5 -> 86.4 mm
- net C3: track 67.2 -> 68.2 mm
- net +12V: track 264.0 -> 263.3 mm
- net C4: track 44.6 -> 45.2 mm
- net C1: track 109.9 -> 109.3 mm
- net SCK: track 14.3 -> 14.8 mm
- net EXP_CS: track 17.1 -> 17.7 mm
- net SDA: track 100.9 -> 100.3 mm
- net GND: vias 66 -> 64
